Commit message: updated naming to match real robot to simplify sim-to-real

File: src/lerobot_description/urdf/so101_base.xacro (robot description, xacro)
@@ -276,5 +276,5 @@
 	</link>
 	<!-- Link gripper -->
-	<link name="gripper">
+	<link name="gripper_link">
 		<inertial>
 			<origin xyz="0.000213627 0.000245138 -0.025187" rpy="0 0 0" />
@@ -340,14 +340,14 @@
 	</link>
 	<!-- Joint from gripper to jaw -->
-	<joint name="6" type="revolute">
+	<joint name="gripper" type="revolute">
 		<origin xyz="0.0202 0.0188 -0.0234" rpy="1.5708 -5.14108e-17 -1.38655e-14" />
-		<parent link="gripper" />
+		<parent link="gripper_link" />
 		<child link="jaw" />
 		<axis xyz="0 0 1" />
 		<limit effort="10" velocity="10" lower="-0.174533" upper="1.74533" />
 	</joint>
-	<transmission name="6_trans">
-		<type>transmission_interface/SimpleTransmission</type>
-		<joint name="6">
+	<transmission name="gripper_trans">
+		<type>transmission_interface/SimpleTransmission</type>
+		<joint name="gripper">
 			<hardwareInterface>hardware_interface/PositionJointInterface</hardwareInterface>
 		</joint>
@@ -358,14 +358,14 @@
 	</transmission>
 	<!-- Joint from wrist to gripper -->
-	<joint name="5" type="revolute">
+	<joint name="wrist_roll" type="revolute">
 		<origin xyz="0 -0.0611 0.0181" rpy="1.5708 -9.38083e-08 3.14159" />
 		<parent link="wrist" />
-		<child link="gripper" />
+		<child link="gripper_link" />
 		<axis xyz="0 0 1" />
 		<limit effort="10" velocity="10" lower="-2.79253" upper="2.79253" />
 	</joint>
-	<transmission name="5_trans">
-		<type>transmission_interface/SimpleTransmission</type>
-		<joint name="5">
+	<transmission name="wrist_roll_trans">
+		<type>transmission_interface/SimpleTransmission</type>
+		<joint name="wrist_roll">
 			<hardwareInterface>hardware_interface/PositionJointInterface</hardwareInterface>
 		</joint>
@@ -376,5 +376,5 @@
 	</transmission>
 	<!-- Joint from lower_arm to wrist -->
-	<joint name="4" type="revolute">
+	<joint name="wrist_flex" type="revolute">
 		<origin xyz="-0.1349 0.0052 1.65232e-16" rpy="3.2474e-15 2.86219e-15 -1.5708" />
 		<parent link="lower_arm" />
@@ -383,7 +383,7 @@
 		<limit effort="10" velocity="10" lower="-1.65806" upper="1.65806" />
 	</joint>
-	<transmission name="4_trans">
-		<type>transmission_interface/SimpleTransmission</type>
-		<joint name="4">
+	<transmission name="wrist_flex_trans">
+		<type>transmission_interface/SimpleTransmission</type>
+		<joint name="wrist_flex">
 			<hardwareInterface>hardware_interface/PositionJointInterface</hardwareInterface>
 		</joint>
@@ -394,5 +394,5 @@
 	</transmission>
 	<!-- Joint from upper_arm to lower_arm -->
-	<joint name="3" type="revolute">
+	<joint name="elbow_flex" type="revolute">
 		<origin xyz="-0.11257 -0.028 2.46331e-16" rpy="-1.22818e-15 5.75928e-16 1.5708" />
 		<parent link="upper_arm" />
@@ -401,7 +401,7 @@
 		<limit effort="10" velocity="10" lower="-1.74533" upper="1.5708" />
 	</joint>
-	<transmission name="3_trans">
-		<type>transmission_interface/SimpleTransmission</type>
-		<joint name="3">
+	<transmission name="elbow_flex_trans">
+		<type>transmission_interface/SimpleTransmission</type>
+		<joint name="elbow_flex">
 			<hardwareInterface>hardware_interface/PositionJointInterface</hardwareInterface>
 		</joint>
@@ -412,5 +412,5 @@
 	</transmission>
 	<!-- Joint from shoulder to upper_arm -->
-	<joint name="2" type="revolute">
+	<joint name="shoulder_lift" type="revolute">
 		<origin xyz="-0.0303992 -0.0182778 -0.0542" rpy="-1.5708 -1.5708 0" />
 		<parent link="shoulder" />
@@ -419,7 +419,7 @@
 		<limit effort="10" velocity="10" lower="-1.74533" upper="1.74533" />
 	</joint>
-	<transmission name="2_trans">
-		<type>transmission_interface/SimpleTransmission</type>
-		<joint name="2">
+	<transmission name="shoulder_lift_trans">
+		<type>transmission_interface/SimpleTransmission</type>
+		<joint name="shoulder_lift">
 			<hardwareInterface>hardware_interface/PositionJointInterface</hardwareInterface>
 		</joint>
@@ -430,5 +430,5 @@
 	</transmission>
 	<!-- Joint from base to shoulder -->
-	<joint name="1" type="revolute">
+	<joint name="shoulder_pan" type="revolute">
 		<origin xyz="0.0207909 -0.0230745 0.0948817" rpy="-3.14159 6.03684e-16 1.5708" />
 		<parent link="base" />
@@ -437,7 +437,7 @@
 		<limit effort="10" velocity="10" lower="-1.91986" upper="1.91986" />
 	</joint>
-	<transmission name="1_trans">
-		<type>transmission_interface/SimpleTransmission</type>
-		<joint name="1">
+	<transmission name="shoulder_pan_trans">
+		<type>transmission_interface/SimpleTransmission</type>
+		<joint name="shoulder_pan">
 			<hardwareInterface>hardware_interface/PositionJointInterface</hardwareInterface>
 		</joint>

File: src/lerobot_description/urdf/so101_ros2_control.xacro (robot description, xacro)
@@ -6,5 +6,5 @@
             <plugin>gz_ros2_control/GazeboSimSystem</plugin>
         </hardware>
-        <joint name="1">
+        <joint name="shoulder_pan">
             <command_interface name="position">
                 <param name="min">-1.91986</param>
@@ -13,5 +13,5 @@
             <state_interface name="position" />
         </joint>
-        <joint name="2">
+        <joint name="shoulder_lift">
             <command_interface name="position">
                 <param name="min">-1.74533</param>
@@ -20,5 +20,5 @@
             <state_interface name="position" />
         </joint>
-        <joint name="3">
+        <joint name="elbow_flex">
             <command_interface name="position">
                 <param name="min">-1.74533</param>
@@ -27,5 +27,5 @@
             <state_interface name="position" />
         </joint>
-        <joint name="4">
+        <joint name="wrist_flex">
             <command_interface name="position">
                 <param name="min">-1.65806</param>
@@ -34,5 +34,5 @@
             <state_interface name="position" />
         </joint>
-        <joint name="5">
+        <joint name="wrist_roll">
             <command_interface name="position">
                 <param name="min">-2.79253</param>
@@ -41,5 +41,5 @@
             <state_interface name="position" />
         </joint>
-        <joint name="6">
+        <joint name="gripper">
             <command_interface name="position">
                 <param name="min">-0.174533</param>
